File: schematics/whammy_kicad/whammy_one_heatsink.kicad_pcb (KiCad board)
At the start: 2 copper layers, 54 parts, among them Q1 2SK2013, Q2 2SJ313, Q3 2SK2013, Q4 2SJ313, U1 OPA2604, U4 4N35, U5 4N35

Commit message: PCB changes
Parts:
- removed R39: 2K2, Resistor_THT:R_Axial_DIN0207_L6.3mm_D2.5mm_P10.16mm_Horizontal
- removed REF** (x4): Heatsink_Fischer_SK104-STC-STIC_35x13mm_2xDrill2.5mm, Heatsink:Heatsink_Fischer_SK104-STC-STIC_35x13mm_2xDrill2.5mm
- moved R16 37.8 mm to (203.2, 83.8), turned to 180 degrees
- moved R32 34.5 mm to (88.9, 83.8), turned to 180 degrees
- moved R6 33.0 mm to (182.9, 101.6)
- moved R22 27.9 mm to (165.1, 83.8), turned to 180 degrees
- moved R29 21.8 mm to (127.0, 83.8), turned to 180 degrees
- moved Q4 20.5 mm to (81.3, 76.2), turned to 0 degrees
- moved U5 20.5 mm to (94.0, 81.3), turned to 0 degrees
- moved R18 19.8 mm to (185.4, 76.2)
- moved R36 18.5 mm to (147.3, 86.4)
- moved R35 18.0 mm to (134.6, 76.2)
- moved R30 17.1 mm to (109.2, 76.2)
- moved C13 17.0 mm to (185.4, 81.3), turned to 270 degrees
- moved R11 16.3 mm to (198.1, 101.6), turned to 90 degrees
- moved C3 15.4 mm to (129.5, 96.5)
- moved C4 15.2 mm to (147.3, 96.5)
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
Commit message: Final version
Parts:
- added C26: 22uF/25V, Capacitor_THT:CP_Radial_D6.3mm_P2.50mm, F.Cu at (181.6, 106.7)
- added C27: 22uF/25V, Capacitor_THT:CP_Radial_D6.3mm_P2.50mm, F.Cu at (97.8, 106.7)
- added J2: Conn_01x03, Connector_JST:JST_EH_B3B-EH-A_1x03_P2.50mm_Vertical, F.Cu at (142.2, 78.7)
- added J3: Conn_01x03, Connector_JST:JST_EH_B3B-EH-A_1x03_P2.50mm_Vertical, F.Cu at (142.2, 121.9)
- added J5: Conn_01x03, Connector_JST:JST_EH_B3B-EH-A_1x03_P2.50mm_Vertical, F.Cu at (142.2, 88.9)
- added REF**: MountingHole_3.2mm_M3_Pad_Via, MountingHole:MountingHole_3.2mm_M3_Pad_Via, F.Cu at (70.0, 125.0)
- added REF**: MountingHole_3.2mm_M3_Pad_Via, MountingHole:MountingHole_3.2mm_M3_Pad_Via, F.Cu at (210.0, 125.0)
- added REF**: MountingHole_3.2mm_M3_Pad_Via, MountingHole:MountingHole_3.2mm_M3_Pad_Via, F.Cu at (210.0, 80.0)
- added REF**: MountingHole_3.2mm_M3_Pad_Via, MountingHole:MountingHole_3.2mm_M3_Pad_Via, F.Cu at (70.0, 80.0)
- moved R1 81.0 mm to (91.4, 105.4)
- moved R12 76.7 mm to (188.0, 105.4), turned to 90 degrees
- moved R26 44.4 mm to (78.7, 91.4)
- moved Q3 39.4 mm to (80.0, 76.2)
- moved R29 37.6 mm to (90.2, 76.2), turned to 0 degrees
- moved Q4 36.8 mm to (118.1, 76.2)
- moved R31 35.8 mm to (118.1, 91.4)
- moved R34 33.3 mm to (123.2, 91.4)
- moved R25 31.5 mm to (82.5, 81.3), turned to 270 degrees
- moved R6 24.7 mm to (196.8, 81.3), turned to 270 degrees
- moved C17 23.9 mm to (176.5, 99.1), turned to 270 degrees
- moved R30 23.4 mm to (86.4, 81.3), turned to 270 degrees
- moved C22 22.5 mm to (102.9, 94.0), turned to 90 degrees
- moved C2 21.6 mm to (78.7, 102.9)
- moved R4 21.6 mm to (86.4, 105.4)
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Routing:
- net +15V: track 0.00 -> 156.5 mm
- net RIGHT_OUT: track 0.00 -> 97.9 mm
- net LEFT_OUT: track 0.00 -> 97.8 mm
- net -15V: track 0.00 -> 73.7 mm
- net Net-(C7-Pad1): track 0.00 -> 60.8 mm
- net Net-(C2-Pad1): track 0.00 -> 59.8 mm
- net Net-(C23-Pad1): track 0.00 -> 49.8 mm
- net Net-(C13-Pad1): track 0.00 -> 44.8 mm
- net Net-(Q4-Pad3): track 0.00 -> 43.4 mm
- net Net-(C12-Pad2): track 0.00 -> 37.9 mm
- net Net-(R5-Pad1): track 0.00 -> 32.1 mm
- net Net-(R2-Pad1): track 0.00 -> 32.1 mm
- net Net-(C22-Pad2): track 0.00 -> 31.9 mm
- net Net-(C4-Pad2): track 0.00 -> 29.5 mm
- net Net-(C22-Pad1): track 0.00 -> 29.0 mm
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- added copper zone on B.Cu, net GND
- added copper zone on F.Cu, net GND
Other:
- board outline added: 150 x 60 mm
